File: ts_foc_fw/EG2134_single_motor/BLDC_driver/BLDC_driver.kicad_sch (KiCad schematic)
At the start: 0 parts

Commit message: 原理图移植完成,PCB还没有布局
Other:
- added sheet Readme (Readme.kicad_sch)
- note added: "Cirrent_sensor"
- note added: "Connection"
- note added: "DC-DC 12/24 -> 5V"
- note added: "EG2134驱动"
- note added: "目录："
Changed lines of the file:
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@@
+		)
+	)
+	(text "DC-DC 12/24 -> 5V"
+		(exclude_from_sim yes)
+		(at 53.594 146.812 0)
+		(effects
+			(font
+				(size 2.54 2.54)
+				(thickness 1.016)
+				(bold yes)
+			)
+			(href "#2")
+		)
+	)
+	(text "EG2134驱动"
+		(exclude_from_sim yes)
+		(at 43.688 153.162 0)
+		(effects
+			(font
+				(size 2.54 2.54)
+				(thickness 1.016)
+				(bold yes)
+			)
+			(href "#3")
+		)
+	)
+	(text "Cirrent_sensor"
+		(exclude_from_sim yes)
+		(at 46.482 163.83 0)
+		(effects
+			(font
+				(size 2.54 2.54)
+				(thickness 1.016)
+				(bold yes)
+			)
+			(href "#5")
 		)
 	)
 	(text "readme:"
 		(exclude_from_sim yes)
-		(at 33.02 22.86 0)
+		(at 30.226 17.78 0)
 		(effects
 			(font
@@
 				(bold yes)
 			)
+			(href "#7")
+		)
+	)
+	(text "目录："
+		(exclude_from_sim yes)
+		(at 24.892 138.176 0)
+		(effects
+			(font
+				(size 3.81 3.81)
+				(thickness 0.4763)
+			)
+		)
+	)
+	(text "Connection\n"
+		(exclude_from_sim yes)
+		(at 43.18 158.75 0)
+		(effects
+			(font
+				(size 2.54 2.54)
+				(thickness 1.016)
+				(bold yes)
+			)
+			(href "#4")
 		)
 	)
@@
 				)
 			)
+		)
+	)
+	(sheet
+		(at 256.54 16.51)
+		(size 26.67 8.89)
+		(fields_autoplaced yes)
+		(stroke
+			(width 0.1524)
+			(type solid)
+		)
+		(fill
+			(color 0 0 0 0.0000)
+		)
+		(property "Sheetname" "Readme"
+			(at 256.54 15.7984 0)
+			(effects
+				(font
+					(size 1.27 1.27)
+				)
+				(justify left bottom)
+			)
+		)
+		(property "Sheetfile" "Readme.kicad_sch"
+			(at 256.54 25.9846 0)
+			(effects
+				(font
+					(size 1.27 1.27)
+				)
+				(justify left top)
+			)
+		)
+		(instances
+			(project "BLDC_driver"
+				(path "/3c13b5e1-57fa-4740-a1aa-c7a3ab53fab1"
+					(page "7")
+				)
+			)
