File: ts_foc_fw/EG2134_single_motor/BLDC_driver/MCU.kicad_sch (KiCad schematic)
At the start: 0 parts

Commit message: PCB_layout_ing
Other:
- note added: "MCU"
Changed lines of the file:
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@@
 	(generator_version "8.0")
 	(paper "A4")
+	(text "MCU"
+		(exclude_from_sim yes)
+		(at 24.13 20.32 0)
+		(effects
+			(font
+				(size 5.08 5.08)
+				(thickness 1.016)
+				(bold yes)
+			)
+			(href "#1")
+		)
+	)
 )
