File: ts_foc_fw/EG2134_single_motor/BLDC_driver/cirrent_sensor.kicad_sch (KiCad schematic)
At the start: 0 parts

Commit message: 原理图移植完成,PCB还没有布局
Parts:
- added R18, R19: res_10r, BLDC_Drive_Tsfoc:R2512, symbol BLDC_Drive_Tsfoc:res_10r
- added U3, U4: INA240A2PW, BLDC_Drive_Tsfoc:INA240A2PW, symbol BLDC_Drive_Tsfoc:INA240A2PW
Connections:
- new net +3.3V: U3.5 (VS), U3.6 (REF2), U4.5 (VS), U4.6 (REF2)
- new net GND: U3.4 (GND), U3.7 (REF1), U4.4 (GND), U4.7 (REF1)
- new net M0_OUT1_CS: U3.8 (OUT)
- new net M0_OUT1_N: R18.2, U3.2 (IN+)
- new net M0_OUT1_P: R18.1, U3.3 (IN-)
- new net M0_OUT2_CS: U4.8 (OUT)
- new net M0_OUT2_N: R19.2, U4.2 (IN+)
- new net M0_OUT2_P: R19.1, U4.3 (IN-)
- no-connect marks 0 -> 2
Other:
- note added: "Connection"

Commit message: PCB_layout_ing
Parts:
- R18, R19: value res_10r -> 10mr
Changed lines of the file:
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@@
 	(wire
 		(pts
-			(xy 64.77 90.17) (xy 69.85 90.17)
-		)
-		(stroke
-			(width 0)
-			(type default)
-		)
-	)
-	(wire
-		(pts
-			(xy 106.68 83.82) (xy 120.65 83.82)
+			(xy 64.77 90.17) (xy 74.93 90.17)
 		)
 		(stroke
@@
 	(wire
 		(pts
-			(xy 74.93 128.27) (xy 64.77 128.27)
+			(xy 64.77 128.27) (xy 74.93 128.27)
 		)
 		(stroke
@@
 	(wire
 		(pts
-			(xy 106.68 132.08) (xy 120.65 132.08)
+			(xy 64.77 80.01) (xy 74.93 80.01)
 		)
 		(stroke
@@
 	(wire
 		(pts
-			(xy 74.93 80.01) (xy 64.77 80.01)
-		)
-		(stroke
-			(width 0)
-			(type default)
-		)
-	)
-	(wire
-		(pts
-			(xy 86.36 88.9) (xy 69.85 88.9)
+			(xy 86.36 88.9) (xy 74.93 88.9)
 		)
 		(stroke
@@
 	(wire
 		(pts
-			(xy 69.85 88.9) (xy 69.85 90.17)
+			(xy 74.93 88.9) (xy 74.93 90.17)
 		)
 		(stroke
@@
 		)
 	)
-	(label "M0_OUT1_CS"
-		(at 109.22 83.82 0)
+	(global_label "M0_OUT2_CS"
+		(shape input)
+		(at 106.68 132.08 0)
 		(fields_autoplaced yes)
 		(effects
@@
 				(size 1.27 1.27)
 			)
-			(justify left bottom)
-		)
-	)
-	(label "M0_OUT1_P"
+			(justify left)
+		)
+		(property "Intersheetrefs" "${INTERSHEET_REFS}"
+			(at 121.5789 132.08 0)
+			(effects
+				(font
+					(size 1.27 1.27)
+				)
+				(justify left)
+				(hide yes)
+			)
+		)
+	)
+	(global_label "M0_OUT1_P"
+		(shape input)
 		(at 64.77 90.17 270)
 		(fields_autoplaced yes)
@@
 				(size 1.27 1.27)
 			)
-			(justify right bottom)
-		)
-	)
-	(label "M0_OUT2_N"
-		(at 64.77 128.27 90)
+			(justify right)
+		)
+		(property "Intersheetrefs" "${INTERSHEET_REFS}"
+			(at 64.77 103.8594 90)
+			(effects
+				(font
+					(size 1.27 1.27)
+				)
+				(justify right)
+				(hide yes)
+			)
+		)
+	)
+	(global_label "M0_OUT1_N"
+		(shape input)
+		(at 64.77 80.01 90)
 		(fields_autoplaced yes)
 		(effects
@@
 				(size 1.27 1.27)
 			)
-			(justify left bottom)
-		)
-	)
-	(label "M0_OUT2_CS"
-		(at 109.22 132.08 0)
+			(justify left)
+		)
+		(property "Intersheetrefs" "${INTERSHEET_REFS}"
+			(at 64.77 66.2601 90)
+			(effects
+				(font
+					(size 1.27 1.27)
+				)
+				(justify left)
+				(hide yes)
+			)
+		)
+	)
+	(global_label "M0_OUT2_N"
+		(shape input)
+		(at 64.77 128.27 90)
 		(fields_autoplaced yes)
 		(effects
@@
 				(size 1.27 1.27)
 			)
-			(justify left bottom)
-		)
-	)
-	(label "M0_OUT2_P"
+			(justify left)
+		)
+		(property "Intersheetrefs" "${INTERSHEET_REFS}"
+			(at 64.77 114.5201 90)
+			(effects
+				(font
+					(size 1.27 1.27)
+				)
+				(justify left)
+				(hide yes)
+			)
+		)
+	)
+	(global_label "M0_OUT2_P"
+		(shape input)
 		(at 64.77 138.43 270)
 		(fields_autoplaced yes)
@@
 				(size 1.27 1.27)
 			)
-			(justify right bottom)
-		)
-	)
-	(label "M0_OUT1_N"
-		(at 64.77 80.01 90)
+			(justify right)
+		)
+		(property "Intersheetrefs" "${INTERSHEET_REFS}"
+			(at 64.77 152.1194 90)
+			(effects
+				(font
+					(size 1.27 1.27)
+				)
+				(justify right)
+				(hide yes)
+			)
+		)
+	)
+	(global_label "M0_OUT1_CS"
+		(shape input)
+		(at 106.68 83.82 0)
 		(fields_autoplaced yes)
 		(effects
@@
 				(size 1.27 1.27)
 			)
-			(justify left bottom)
+			(justify left)
+		)
+		(property "Intersheetrefs" "${INTERSHEET_REFS}"
+			(at 121.5789 83.82 0)
+			(effects
+				(font
+					(size 1.27 1.27)
+				)
+				(justify left)
+				(hide yes)
+			)
 		)
 	)
@@
 			)
 		)
-		(property "Value" "res_10r"
+		(property "Value" "10mr"
 			(at 67.31 134.6199 90)
 			(effects
@@
 			)
 		)
-		(property "Value" "res_10r"
+		(property "Value" "10mr"
 			(at 67.31 86.3599 90)
 			(effects
