File: ts_foc_fw/EG2134_single_motor/EG2134_single_motor_drive/Power.kicad_sch (KiCad schematic)
At the start: 18 parts, among them U1 SY8205FCC

Commit message: PCB布局完成，等待布线
Parts:
- added TP2_VCC1: VCC, TestPoint:TestPoint_Pad_D1.5mm, symbol Connector:TestPoint
- renumbered C6 to C10, C5 to C11, C4 to C12, C3 to C13, C2 to C14, C1 to C15, C10 to C6, C9 to C7, C7 to C9, R4 to R13, R2 to R14, R3 to R15, R1 to R16, TP1 to TP1_3V1, U1 to U2
Connections:
- net VCC: now also TP2_VCC1.1
Changed lines of the file:
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@@
+	)
+	(junction
+		(at 222.25 105.41)
+		(diameter 0)
+		(color 0 0 0 0)
 	)
 	(junction
@@
 	(wire
 		(pts
-			(xy 214.63 105.41) (xy 209.55 105.41)
+			(xy 226.06 105.41) (xy 222.25 105.41)
 		)
 		(stroke
@@
 		(pts
 			(xy 185.42 110.49) (xy 184.15 110.49)
+		)
+		(stroke
+			(width 0)
+			(type default)
+		)
+	)
+	(wire
+		(pts
+			(xy 222.25 105.41) (xy 209.55 105.41)
 		)
 		(stroke
@@
 		(on_board yes)
 		(dnp no)
-		(property "Reference" "C1"
+		(property "Reference" "C15"
 			(at 204.47 103.886 0)
 			(effects
@@
 			(project "EG2134_single_motor_drive"
 				(path "/a69a3027-f6f2-4dc7-8446-d1a07c691b27/c784a5b9-792f-4178-b63e-bae01c34cf3b"
-					(reference "C1")
+					(reference "C15")
 					(unit 1)
 				)
@@
 		(dnp no)
 		(fields_autoplaced yes)
-		(property "Reference" "U1"
+		(property "Reference" "U2"
 			(at 171.45 95.25 0)
 			(effects
@@
 			(project ""
 				(path "/a69a3027-f6f2-4dc7-8446-d1a07c691b27/c784a5b9-792f-4178-b63e-bae01c34cf3b"
-					(reference "U1")
+					(reference "U2")
 					(unit 1)
 				)
@@
 		(dnp no)
 		(fields_autoplaced yes)
-		(property "Reference" "R1"
+		(property "Reference" "R16"
 			(at 212.09 99.0599 90)
 			(effects
@@
 			(project ""
 				(path "/a69a3027-f6f2-4dc7-8446-d1a07c691b27/c784a5b9-792f-4178-b63e-bae01c34cf3b"
-					(reference "R1")
+					(reference "R16")
 					(unit 1)
 				)
@@
 		(on_board yes)
 		(dnp no)
-		(property "Reference" "#PWR04"
+		(property "Reference" "#PWR016"
 			(at 156.21 127 0)
 			(effects
@@
 			(project "EG2134_single_motor_drive"
 				(path "/a69a3027-f6f2-4dc7-8446-d1a07c691b27/c784a5b9-792f-4178-b63e-bae01c34cf3b"
-					(reference "#PWR04")
+					(reference "#PWR016")
 					(unit 1)
 				)
@@
 		(on_board yes)
 		(dnp no)
-		(property "Reference" "#PWR05"
+		(property "Reference" "#PWR015"
 			(at 129.54 135.89 0)
 			(effects
@@
 			(project "EG2134_single_motor_drive"
 				(path "/a69a3027-f6f2-4dc7-8446-d1a07c691b27/c784a5b9-792f-4178-b63e-bae01c34cf3b"
-					(reference "#PWR05")
+					(reference "#PWR015")
 					(unit 1)
 				)
@@
 		(dnp no)
 		(fields_autoplaced yes)
-		(property "Reference" "R2"
+		(property "Reference" "R14"
 			(at 132.08 109.2199 90)
 			(effects
@@
 			(project "EG2134_single_motor_drive"
 				(path "/a69a3027-f6f2-4dc7-8446-d1a07c691b27/c784a5b9-792f-4178-b63e-bae01c34cf3b"
-					(reference "R2")
+					(reference "R14")
 					(unit 1)
 				)
@@
 		(on_board yes)
 		(dnp no)
-		(property "Reference" "#PWR08"
+		(property "Reference" "#PWR012"
 			(at 83.82 113.03 0)
 			(effects
@@
 			(project "EG2134_single_motor_drive"
 				(path "/a69a3027-f6f2-4dc7-8446-d1a07c691b27/c784a5b9-792f-4178-b63e-bae01c34cf3b"
-					(reference "#PWR08")
+					(reference "#PWR012")
 					(unit 1)
 				)
@@
 	(symbol
 		(lib_id "power:VCC")
-		(at 214.63 105.41 270)
+		(at 226.06 105.41 270)
 		(unit 1)
 		(exclude_from_sim no)
@@
 		(dnp no)
 		(fields_autoplaced yes)
-		(property "Reference" "#PWR01"
-			(at 210.82 105.41 0)
+		(property "Reference" "#PWR019"
+			(at 222.25 105.41 0)
 			(effects
 				(font
@@
 		)
 		(property "Value" "VCC"
-			(at 218.44 105.4099 90)
+			(at 229.87 105.4099 90)
 			(effects
 				(font
@@
 		)
 		(property "Footprint" ""
-			(at 214.63 105.41 0)
+			(at 226.06 105.41 0)
 			(effects
 				(font
@@
 		)
 		(property "Datasheet" ""
-			(at 214.63 105.41 0)
+			(at 226.06 105.41 0)
 			(effects
 				(font
@@
 		)
 		(property "Description" "Power symbol creates a global label with name \"VCC\""
-			(at 214.63 105.41 0)
+			(at 226.06 105.41 0)
 			(effects
 				(font
@@
 			(project "EG2134_single_motor_drive"
 				(path "/a69a3027-f6f2-4dc7-8446-d1a07c691b27/c784a5b9-792f-4178-b63e-bae01c34cf3b"
-					(reference "#PWR01")
+					(reference "#PWR019")
 					(unit 1)
 				)
@@
 		(on_board yes)
 		(dnp no)
-		(property "Reference" "C9"
+		(property "Reference" "C7"
 			(at 114.3 114.046 0)
 			(effects
@@
 			(project "EG2134_single_motor_drive"
 				(path "/a69a3027-f6f2-4dc7-8446-d1a07c691b27/c784a5b9-792f-4178-b63e-bae01c34cf3b"
-					(reference "C9")
+					(reference "C7")
 					(unit 1)
 				)
@@
 		(dnp no)
 		(fields_autoplaced yes)
-		(property "Reference" "R3"
+		(property "Reference" "R15"
 			(at 132.08 123.1899 90)
 			(effects
@@
 			(project "EG2134_single_motor_drive"
 				(path "/a69a3027-f6f2-4dc7-8446-d1a07c691b27/c784a5b9-792f-4178-b63e-bae01c34cf3b"
-					(reference "R3")
+					(reference "R15")
 					(unit 1)
 				)
@@
 		(on_board yes)
 		(dnp no)
-		(property "Reference" "C6"
+		(property "Reference" "C10"
 			(at 157.226 101.6 0)
 			(effects
@@
 			(project "EG2134_single_motor_drive"
 				(path "/a69a3027-f6f2-4dc7-8446-d1a07c691b27/c784a5b9-792f-4178-b63e-bae01c34cf3b"
-					(reference "C6")
+					(reference "C10")
 					(unit 1)
 				)
@@
 		(dnp no)
 		(fields_autoplaced yes)
-		(property "Reference" "#PWR02"
+		(property "Reference" "#PWR018"
 			(at 204.47 110.49 0)
 			(effects
@@
 			(project "EG2134_single_motor_drive"
 				(path "/a69a3027-f6f2-4dc7-8446-d1a07c691b27/c784a5b9-792f-4178-b63e-bae01c34cf3b"
-					(reference "#PWR02")
+					(reference "#PWR018")
 					(unit 1)
 				)
@@
 		(on_board yes)
 		(dnp no)
-		(property "Reference" "C5"
+		(property "Reference" "C11"
 			(at 157.48 119.126 0)
 			(effects
@@
 			(project "EG2134_single_motor_drive"
 				(path "/a69a3027-f6f2-4dc7-8446-d1a07c691b27/c784a5b9-792f-4178-b63e-bae01c34cf3b"
-					(reference "C5")
+					(reference "C11")
 					(unit 1)
 				)
@@
 		(on_board yes)
 		(dnp no)
-		(property "Reference" "TP1"
+		(property "Reference" "TP1_3V1"
 			(at 109.728 100.076 0)
 			(effects
@@
 			(project ""
 				(path "/a69a3027-f6f2-4dc7-8446-d1a07c691b27/c784a5b9-792f-4178-b63e-bae01c34cf3b"
-					(reference "TP1")
+					(reference "TP1_3V1")
 					(unit 1)
 				)
@@
 		(dnp no)
 		(fields_autoplaced yes)
-		(property "Reference" "#PWR03"
+		(property "Reference" "#PWR017"
 			(at 187.96 85.09 0)
 			(effects
@@
 			(project "EG2134_single_motor_drive"
 				(path "/a69a3027-f6f2-4dc7-8446-d1a07c691b27/c784a5b9-792f-4178-b63e-bae01c34cf3b"
-					(reference "#PWR03")
+					(reference "#PWR017")
 					(unit 1)
 				)
@@
 		(on_board yes)
 		(dnp no)
-		(property "Reference" "C4"
+		(property "Reference" "C12"
 			(at 194.056 109.22 0)
 			(effects
@@
 			(project "EG2134_single_motor_drive"
 				(path "/a69a3027-f6f2-4dc7-8446-d1a07c691b27/c784a5b9-792f-4178-b63e-bae01c34cf3b"
-					(reference "C4")
+					(reference "C12")
 					(unit 1)
 				)
@@
 		(dnp no)
 		(fields_autoplaced yes)
-		(property "Reference" "R4"
+		(property "Reference" "R13"
 			(at 99.06 99.06 0)
 			(effects
@@
 			(project "EG2134_single_motor_drive"
 				(path "/a69a3027-f6f2-4dc7-8446-d1a07c691b27/c784a5b9-792f-4178-b63e-bae01c34cf3b"
-					(reference "R4")
+					(reference "R13")
 					(unit 1)
 				)
@@
 		(dnp no)
 		(fields_autoplaced yes)
-		(property "Reference" "#PWR07"
+		(property "Reference" "#PWR014"
 			(at 107.95 104.14 0)
 			(effects
@@
 			(project ""
 				(path "/a69a3027-f6f2-4dc7-8446-d1a07c691b27/c784a5b9-792f-4178-b63e-bae01c34cf3b"
-					(reference "#PWR07")
+					(reference "#PWR014")
 					(unit 1)
 				)
@@
 		(on_board yes)
 		(dnp no)
-		(property "Reference" "C10"
+		(property "Reference" "C6"
 			(at 109.22 114.046 0)
 			(effects
@@
 			(project "EG2134_single_motor_drive"
 				(path "/a69a3027-f6f2-4dc7-8446-d1a07c691b27/c784a5b9-792f-4178-b63e-bae01c34cf3b"
-					(reference "C10")
+					(reference "C6")
+					(unit 1)
+				)
+			)
+		)
+	)
+	(symbol
+		(lib_id "Connector:TestPoint")
+		(at 222.25 105.41 180)
+		(unit 1)
+		(exclude_from_sim no)
+		(in_bom yes)
+		(on_board yes)
+		(dnp no)
+		(property "Reference" "TP2_VCC1"
+			(at 223.012 110.744 0)
+			(effects
+				(font
+					(size 1.27 1.27)
+				)
+				(justify left)
+			)
+		)
+		(property "Value" "VCC"
+			(at 221.234 108.458 0)
+			(effects
+				(font
+					(size 1.27 1.27)
+				)
+				(justify left)
+			)
+		)
+		(property "Footprint" "TestPoint:TestPoint_Pad_D1.5mm"
+			(at 217.17 105.41 0)
+			(effects
+				(font
+					(size 1.27 1.27)
+				)
+				(hide yes)
+			)
+		)
+		(property "Datasheet" "~"
+			(at 217.17 105.41 0)
+			(effects
+				(font
+					(size 1.27 1.27)
+				)
+				(hide yes)
+			)
+		)
+		(property "Description" "test point"
+			(at 222.25 105.41 0)
+			(effects
+				(font
+					(size 1.27 1.27)
+				)
+				(hide yes)
+			)
+		)
+		(pin "1"
+		)
+		(instances
+			(project "EG2134_single_motor_drive"
+				(path "/a69a3027-f6f2-4dc7-8446-d1a07c691b27/c784a5b9-792f-4178-b63e-bae01c34cf3b"
+					(reference "TP2_VCC1")
 					(unit 1)
 				)
@@
 		(on_board yes)
 		(dnp no)
-		(property "Reference" "C7"
+		(property "Reference" "C9"
 			(at 125.73 114.046 0)
 			(effects
@@
 			(project "EG2134_single_motor_drive"
 				(path "/a69a3027-f6f2-4dc7-8446-d1a07c691b27/c784a5b9-792f-4178-b63e-bae01c34cf3b"
-					(reference "C7")
+					(reference "C9")
 					(unit 1)
 				)
@@
 		(on_board yes)
 		(dnp no)
-		(property "Reference" "C2"
+		(property "Reference" "C14"
 			(at 199.39 103.886 0)
 			(effects
@@
 			(project "EG2134_single_motor_drive"
 				(path "/a69a3027-f6f2-4dc7-8446-d1a07c691b27/c784a5b9-792f-4178-b63e-bae01c34cf3b"
-					(reference "C2")
+					(reference "C14")
 					(unit 1)
 				)
@@
 		(on_board yes)
 		(dnp no)
-		(property "Reference" "#PWR06"
+		(property "Reference" "#PWR013"
 			(at 90.17 115.57 0)
 			(effects
@@
 			(project "EG2134_single_motor_drive"
 				(path "/a69a3027-f6f2-4dc7-8446-d1a07c691b27/c784a5b9-792f-4178-b63e-bae01c34cf3b"
-					(reference "#PWR06")
+					(reference "#PWR013")
 					(unit 1)
 				)
@@
 		(on_board yes)
 		(dnp no)
-		(property "Reference" "C3"
+		(property "Reference" "C13"
 			(at 194.31 103.886 0)
 			(effects
@@
 			(project "EG2134_single_motor_drive"
 				(path "/a69a3027-f6f2-4dc7-8446-d1a07c691b27/c784a5b9-792f-4178-b63e-bae01c34cf3b"
-					(reference "C3")
-					(unit 1)
-				)
+					(reference "C13")
+					(unit 1)
+				)
