File: ts_foc_fw/EG2134_single_motor/EG2134_single_motor_drive/EG2134_single_motor_drive.kicad_pcb (KiCad board)
At the start: 4 copper layers, 61.3 x 22.9 mm, 61 parts, among them CN1 XT30PW-M, CN2 WAFER-GH1.25-10PWB, Q1 RU3089M-C, Q2 RU3089M-C, Q3 RU3089M-C, Q4 RU3089M-C, Q5 RU3089M-C, Q6 RU3089M-C, U1 EG2134_N, U2 SY8205FCC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

Commit message: tongbu
Connections:
- CN2 pad 6: CS_2 -> CS2
- CN2 pad 7: CS_1 -> CS1
Routing:
- net CS1: track 0.00 -> 18.0 mm, vias 0 -> 2
- net CS2: track 0.00 -> 13.4 mm
- net GND: track 24.1 -> 29.1 mm
