File: ts_foc_fw/Ts_Foc_Vo1.0/Ts_Foc_Vo1_0/Ts_Foc_Vo1_0.kicad_sch (KiCad schematic)
At the start: 0 parts

Commit message: 同步_Fri Jan 24 20:31:29     2025
Other:
- added sheet Connector (Connector.kicad_sch)
- added sheet Drive (Drive.kicad_sch)
- added sheet Mcu (Mcu.kicad_sch)
- added sheet Power (Power.kicad_sch)
- note added: "1.本项目根据Ts_Foc单电机版本迭代"
- note added: "2.布局参考odriver3.6开源版本"
- note added: "3."
- note added: "Readme:"
