File: TsFoc/ts_foc_fw/Ts_Foc_Vo1.0/Ts_Foc_Vo1_0/Connector.kicad_sch (KiCad schematic)
At the start: 13 parts, among them CN1 MR30PW-M30.G.Y, CN10 GH1.25-4P, CN11 GH1.25-5PLT, CN12 GH1.25-5PLT, CN2 MR30PW-M30.G.Y, CN3 GH1.25-2P_LT, CN4 GH1.25-2P_LT, CN5 XT30PW-M, CN6 GH1.25-4P, CN7 GH1.25-4P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

Commit message: vscode尝试同步
Parts:
- added TV1: SMAJ36CA, Ts_Foc_Vo封装库:SMA_L4.4, symbol Ts_Foc_Vo符号库:SMAJ36CA
Connections:
- net GND: now also TV1.1 (K)
- net UART2-RX: no longer CN8.2
- net UART2-TX: no longer CN8.1
- net VCC: now also TV1.2 (A)
- new net UART3-RX: CN8.2
- new net UART3-TX: CN8.1
Changed lines of the file:
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@@
 		(rev "Dennis_Re_Yoonjiho")
 	)
+	(junction
+		(at 129.54 43.18)
+		(diameter 0)
+		(color 0 0 0 0)
+	)
+	(junction
+		(at 129.54 33.02)
+		(diameter 0)
+		(color 0 0 0 0)
+	)
+	(wire
+		(pts
+			(xy 137.16 38.1) (xy 140.97 38.1)
+		)
+		(stroke
+			(width 0)
+			(type default)
+		)
+	)
+	(wire
+		(pts
+			(xy 127 33.02) (xy 129.54 33.02)
+		)
+		(stroke
+			(width 0)
+			(type default)
+		)
+	)
+	(wire
+		(pts
+			(xy 129.54 43.18) (xy 137.16 43.18)
+		)
+		(stroke
+			(width 0)
+			(type default)
+		)
+	)
+	(wire
+		(pts
+			(xy 137.16 40.64) (xy 140.97 40.64)
+		)
+		(stroke
+			(width 0)
+			(type default)
+		)
+	)
+	(wire
+		(pts
+			(xy 137.16 33.02) (xy 137.16 38.1)
+		)
+		(stroke
+			(width 0)
+			(type default)
+		)
+	)
+	(wire
+		(pts
+			(xy 127 43.18) (xy 129.54 43.18)
+		)
+		(stroke
+			(width 0)
+			(type default)
+		)
+	)
+	(wire
+		(pts
+			(xy 137.16 43.18) (xy 137.16 40.64)
+		)
+		(stroke
+			(width 0)
+			(type default)
+		)
+	)
+	(wire
+		(pts
+			(xy 129.54 33.02) (xy 137.16 33.02)
+		)
+		(stroke
+			(width 0)
+			(type default)
+		)
+	)
 	(text "CAN\n"
 		(exclude_from_sim yes)
@@
 		)
 	)
-	(global_label "UART2-TX"
+	(global_label "UART3-TX"
 		(shape bidirectional)
 		(at 85.09 115.57 180)
@@
 		)
 	)
-	(global_label "UART2-RX"
+	(global_label "UART3-RX"
 		(shape bidirectional)
 		(at 85.09 118.11 180)
@@
 	(symbol
 		(lib_id "power:GND")
-		(at 140.97 40.64 270)
+		(at 127 43.18 270)
 		(unit 1)
 		(exclude_from_sim no)
@@
 		(dnp no)
 		(property "Reference" "#PWR057"
-			(at 134.62 40.64 0)
+			(at 120.65 43.18 0)
 			(effects
 				(font
@@
 		)
 		(property "Value" "GND"
-			(at 137.414 40.64 0)
+			(at 123.444 43.18 0)
 			(effects
 				(font
@@
 		)
 		(property "Footprint" ""
-			(at 140.97 40.64 0)
+			(at 127 43.18 0)
 			(effects
 				(font
@@
 		)
 		(property "Datasheet" ""
-			(at 140.97 40.64 0)
+			(at 127 43.18 0)
 			(effects
 				(font
@@
 		)
 		(property "Description" "Power symbol creates a global label with name \"GND\" , ground"
-			(at 140.97 40.64 0)
+			(at 127 43.18 0)
 			(effects
 				(font
@@
 	(symbol
 		(lib_id "power:VCC")
-		(at 140.97 38.1 90)
+		(at 127 33.02 90)
 		(unit 1)
 		(exclude_from_sim no)
@@
 		(fields_autoplaced yes)
 		(property "Reference" "#PWR056"
-			(at 144.78 38.1 0)
+			(at 130.81 33.02 0)
 			(effects
 				(font
@@
 		)
 		(property "Value" "VCC"
-			(at 137.16 38.0999 90)
+			(at 123.19 33.0199 90)
 			(effects
 				(font
@@
 		)
 		(property "Footprint" ""
-			(at 140.97 38.1 0)
+			(at 127 33.02 0)
 			(effects
 				(font
@@
 		)
 		(property "Datasheet" ""
-			(at 140.97 38.1 0)
+			(at 127 33.02 0)
 			(effects
 				(font
@@
 		)
 		(property "Description" "Power symbol creates a global label with name \"VCC\""
-			(at 140.97 38.1 0)
+			(at 127 33.02 0)
 			(effects
 				(font
@@
 					(unit 1)
 				)
+			)
+		)
+	)
+	(symbol
+		(lib_id "Ts_Foc_Vo符号库:SMAJ36CA")
+		(at 129.54 38.1 90)
+		(unit 1)
+		(exclude_from_sim no)
+		(in_bom yes)
+		(on_board yes)
+		(dnp no)
+		(fields_autoplaced yes)
+		(property "Reference" "TV1"
+			(at 132.08 36.8299 90)
+			(effects
+				(font
+					(size 1.27 1.27)
+				)
+				(justify right)
+			)
+		)
+		(property "Value" "SMAJ36CA"
+			(at 132.08 39.3699 90)
+			(effects
+				(font
+					(size 1.27 1.27)
+				)
+				(justify right)
+			)
+		)
+		(property "Footprint" "Ts_Foc_Vo封装库:SMA_L4.4"
+			(at 130.81 38.1 0)
+			(effects
+				(font
+					(size 1.27 1.27)
+				)
+				(hide yes)
+			)
+		)
+		(property "Datasheet" "http://www.szlcsc.com/product/details_88448.html"
+			(at 135.89 38.1 0)
+			(effects
+				(font
+					(size 1.27 1.27)
+				)
+				(hide yes)
+			)
+		)
+		(property "Description" ""
+			(at 129.54 38.1 0)
+			(effects
+				(font
+					(size 1.27 1.27)
+				)
+				(hide yes)
+			)
+		)
+		(property "SuppliersPartNumber" "C87270"
+			(at 140.97 38.1 0)
+			(effects
+				(font
+					(size 1.27 1.27)
+				)
+				(hide yes)
+			)
+		)
+		(property "uuid" "std:080b688eba436c70954d860205d81b8f"
+			(at 140.97 38.1 0)
+			(effects
+				(font
+					(size 1.27 1.27)
+				)
+				(hide yes)
+			)
+		)
+		(pin "1"
+		)
+		(pin "2"
+		)
+		(instances
+			(project ""
+				(path "/0cbcabec-8024-48c7-ab91-86e279a5637e/f3329442-eac4-40be-b987-eebdbe922017"
+					(reference "TV1")
+					(unit 1)
+				)
