File: TsFoc/ts_foc_fw/Ts_Foc_Vo1.0/Ts_Foc_Vo1_0/12-5V.kicad_sch (KiCad schematic)
At the start: 12 parts, among them U1 TPS5430DDAR

Commit message: 同步_原理图小幅优化
Other:
- moved on the sheet: C1, C2, C3, C4, C5, C6, D1, L1, R1, R2, R3, U1
