File: TsFoc/ts_foc_fw/Ts_Foc_Vo1.0/Ts_Foc_Vo1_0/5-3V3.kicad_sch (KiCad schematic)
At the start: 5 parts, among them U2 AMS1117-3.3V

Commit message: 同步_原理图小幅优化
Other:
- moved on the sheet: C10, C7, C8, C9, U2
