File: TsFoc/ts_foc_fw/Ts_Foc_Vo1.0/Ts_Foc_Vo1_0/Ts_Foc_Vo1_0.kicad_pcb (KiCad board)
At the start: 2 copper layers, 129 parts, among them CN1 MR30PW-M30.G.Y, CN10 GH1.25-4P, CN11 GH1.25-5PLT, CN12 GH1.25-5PLT, CN2 MR30PW-M30.G.Y, CN3 GH1.25-2P_LT, CN4 GH1.25-2P_LT, CN5 XT30PW-M, CN6 GH1.25-4P, CN7 GH1.25-4P, CN8 GH1.25-4P, CN9 GH1.25-4P, J1 Conn_01x04, Q1 JSM2301S, Q10 RU3089M-C, Q11 RU3089M-C, Q12 RU3089M-C, Q13 RU3089M-C, Q2 RU3089M-C, Q3 RU3089M-C, Q4 RU3089M-C, Q5 RU3089M-C, Q6 RU3089M-C, Q7 RU3089M-C, Q8 RU3089M-C, Q9 RU3089M-C, SW1 BOTTOM, SW2 BOTTOM, U1 TPS5430DDAR, U10 SIT1050TK, U11 SIT1050TK, U2 AMS1117-3.3V, U3 STM32F407VET6, U4 EG2133, U5 INA240A2PWR, U6 INA240A2PWR, U7 EG2133, U8 INA240A2PWR, U9 INA240A2PWR, X1 25Mhz

Commit message: vscode尝试同步
Parts:
- added TV1: SMAJ36CA, Ts_Foc_Vo封装库:SMA_L4.4, F.Cu at (19.4, 42.2)
- moved CN9 81.5 mm to (68.1, 55.2), turned to 180 degrees
- moved CN10 72.1 mm to (58.9, 55.1), turned to 180 degrees
- moved CN11 63.6 mm to (85.8, -17.6)
- moved R33 49.2 mm to (42.0, -22.0)
- moved R34 49.2 mm to (42.0, -19.9)
- moved R35 49.2 mm to (42.0, -17.7)
- moved R36 49.2 mm to (42.0, -15.6)
- moved USB1 49.2 mm to (35.1, -19.6)
- moved C24 41.0 mm to (60.0, 27.6)
- moved C25 41.0 mm to (60.0, 29.8)
- moved C26 41.0 mm to (60.0, 31.9)
- moved C27 40.9 mm to (60.1, 33.9)
- moved C28 40.9 mm to (60.1, 36.2)
- moved D12 39.1 mm to (48.2, 28.8)
- moved D13 39.1 mm to (48.2, 31.7)
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Connections:
- CN8 pad 1: UART2-TX -> UART3-TX
- CN8 pad 2: UART2-RX -> UART3-RX

Commit message: 同步_原理图小幅优化
Connections:
- R12 pad 1: RGB-G -> Net-(LED3-R-)
- R12 pad 2: Net-(LED3-G-) -> RGB-R
- R13 pad 1: RGB-B -> RGB-G
- R13 pad 2: Net-(LED3-B-) -> Net-(LED3-G-)
- R14 pad 1: Net-(LED3-R-) -> RGB-B
- R14 pad 2: RGB-R -> Net-(LED3-B-)
Changed lines of the file:
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@@
 			(size 0.566 0.54)
 			(layers "F.Cu" "F.Paste" "F.Mask")
-			(net 33 "RGB-B")
+			(net 32 "RGB-G")
 			(pinfunction "1")
 			(pintype "input")
@@
 			(size 0.566 0.54)
 			(layers "F.Cu" "F.Paste" "F.Mask")
-			(net 24 "Net-(LED3-B-)")
+			(net 26 "Net-(LED3-G-)")
 			(pinfunction "2")
 			(pintype "input")
@@
 			(size 0.566 0.54)
 			(layers "F.Cu" "F.Paste" "F.Mask")
-			(net 25 "Net-(LED3-R-)")
+			(net 33 "RGB-B")
 			(pinfunction "1")
 			(pintype "input")
@@
 			(size 0.566 0.54)
 			(layers "F.Cu" "F.Paste" "F.Mask")
-			(net 34 "RGB-R")
+			(net 24 "Net-(LED3-B-)")
 			(pinfunction "2")
 			(pintype "input")
@@
 			(size 0.566 0.54)
 			(layers "F.Cu" "F.Paste" "F.Mask")
-			(net 32 "RGB-G")
+			(net 25 "Net-(LED3-R-)")
 			(pinfunction "1")
 			(pintype "input")
@@
 			(size 0.566 0.54)
 			(layers "F.Cu" "F.Paste" "F.Mask")
-			(net 26 "Net-(LED3-G-)")
+			(net 34 "RGB-R")
 			(pinfunction "2")
 			(pintype "input")
