File: TsFoc/ts_foc_fw/Ts_Foc_Vo1.0/Ts_Foc_Vo1_0/drive2.kicad_sch (KiCad schematic)
At the start: 31 parts, among them Q10 RU3089M-C, Q11 RU3089M-C, Q12 RU3089M-C, Q13 RU3089M-C, Q8 RU3089M-C, Q9 RU3089M-C, U7 EG2133, U8 INA240A2PWR, U9 INA240A2PWR

Commit message: 同步_原理图小幅优化
Other:
- note added: "Motor2"
- note removed: "Motor1"
Changed lines of the file:
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@@
 		)
 	)
-	(text "Motor1\n"
+	(text "Motor2"
 		(exclude_from_sim yes)
 		(at 204.978 33.02 0)
