File: TsFoc/ts_foc_fw/Ts_Foc_Vesc0.1/Ts_Foc_Vesc0_1/drive1.kicad_sch (KiCad schematic)
At the start: 31 parts, among them Q2 RU3089M-C, Q3 RU3089M-C, Q4 RU3089M-C, Q5 RU3089M-C, Q6 RU3089M-C, Q7 RU3089M-C, U4 EG2133, U5 INA240A2PWR, U6 INA240A2PWR

Commit message: PCB_Layout_success
Connections:
- net 5V: now also C19.2, C20.2, U4.7 (VCC)
Changed lines of the file:
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@@
+		)
+	)
+	(global_label "5V"
+		(shape bidirectional)
+		(at 34.29 67.31 90)
+		(fields_autoplaced yes)
+		(effects
+			(font
+				(size 1.27 1.27)
+			)
+			(justify left)
+		)
+		(property "Intersheetrefs" "${INTERSHEET_REFS}"
+			(at 34.29 60.9154 90)
+			(effects
+				(font
+					(size 1.27 1.27)
+				)
+				(justify left)
+				(hide yes)
+			)
 		)
 	)
