File: TsFoc/ts_foc_fw/Ts_Foc_Vesc0.1/Ts_Foc_Vesc0_1/drive2.kicad_sch (KiCad schematic)
At the start: 31 parts, among them Q10 RU3089M-C, Q11 RU3089M-C, Q12 RU3089M-C, Q13 RU3089M-C, Q8 RU3089M-C, Q9 RU3089M-C, U7 EG2133, U8 INA240A2PWR, U9 INA240A2PWR

Commit message: PCB_Layout_success
Connections:
- net 5V: now also C24.2, C25.2, U7.7 (VCC)
Changed lines of the file:
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@@
+		)
+	)
+	(global_label "5V"
+		(shape bidirectional)
+		(at 33.02 67.31 90)
+		(fields_autoplaced yes)
+		(effects
+			(font
+				(size 1.27 1.27)
+			)
+			(justify left)
+		)
+		(property "Intersheetrefs" "${INTERSHEET_REFS}"
+			(at 33.02 60.9154 90)
+			(effects
+				(font
+					(size 1.27 1.27)
+				)
+				(justify left)
+				(hide yes)
+			)
 		)
 	)
