File: TsFoc/ts_foc_fw/Ts_Foc_Vesc0.1/Ts_Foc_Vesc0_1/Power.kicad_sch (KiCad schematic)
At the start: 5 parts, among them Q1 JSM2301S

Commit message: PCB_Layout_success
Connections:
- net 5V_USB renamed 5V-USB
Changed lines of the file:
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@@
 		)
 	)
-	(global_label "5V_USB"
+	(global_label "5V-USB"
 		(shape input)
 		(at 179.07 57.15 180)
@@
 		)
 		(property "Intersheetrefs" "${INTERSHEET_REFS}"
-			(at 169.0091 57.15 0)
+			(at 168.4043 57.15 0)
 			(effects
 				(font

Commit message: 电源走线完成
Parts:
- added R38: 0r, Ts_Foc_Vo封装库:Res_0402, symbol Ts_Foc_Vo符号库:RES
Connections:
- net GND: now also R38.1
- new net PGND: R38.2
Other:
- moved on the sheet: LED1, R4
