File: TsFoc/ts_foc_fw/Ts_Foc_Vesc0.1/Ts_Foc_Vesc0_1/STM32F407VET6.kicad_sch (KiCad schematic)
At the start: 15 parts, among them SW2 BOTTOM, U3 STM32F407VET6, X1 25Mhz

Commit message: PCB_Layout_success
Parts:
- added C32, C33, C34, C35, C36, C37, C38, C39, C40, C41, C42: 100nf, Ts_Foc_Vo封装库:CAP_0402, symbol Ts_Foc_Vo符号库:CAP
Connections:
- net 3V3: now also C32.1, C33.1, C34.1, C35.1, C36.1, C37.1, C38.1, C39.1, C40.1, C41.1, C42.1
- net GND: now also C32.2, C33.2, C34.2, C35.2, C36.2, C37.2, C38.2, C39.2, C40.2, C41.2, C42.2

Commit message: 电源走线完成
Connections:
- net USB-DM renamed USB-DN
Changed lines of the file:
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@@
 		)
 	)
-	(global_label "USB-DM"
+	(global_label "USB-DN"
 		(shape bidirectional)
 		(at 48.26 54.61 180)
@@
 		)
 		(property "Intersheetrefs" "${INTERSHEET_REFS}"
-			(at 36.0597 54.61 0)
+			(at 36.1806 54.61 0)
 			(effects
 				(font
