File: TsFoc/ts_foc_fw/Ts_Foc_Vesc0.1/Ts_Foc_Vesc0_1/USB.kicad_sch (KiCad schematic)
At the start: 5 parts

Commit message: PCB_Layout_success
Parts:
- added R37: 1.5k, Ts_Foc_Vo封装库:Res_0402, symbol Ts_Foc_Vo符号库:RES
Connections:
- net DP: now also R37.2
- new net 3V3: R37.1
Changed lines of the file:
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@@
+		)
+	)
+	(global_label "3V3"
+		(shape bidirectional)
+		(at 148.59 148.59 180)
+		(fields_autoplaced yes)
+		(effects
+			(font
+				(size 1.27 1.27)
+			)
+			(justify right)
+		)
+		(property "Intersheetrefs" "${INTERSHEET_REFS}"
+			(at 140.9859 148.59 0)
+			(effects
+				(font
+					(size 1.27 1.27)
+				)
+				(justify right)
+				(hide yes)
+			)
 		)
 	)
@@
 				)
 				(justify right)
+				(hide yes)
+			)
+		)
+	)
+	(global_label "DP"
+		(shape bidirectional)
+		(at 158.75 148.59 0)
+		(fields_autoplaced yes)
+		(effects
+			(font
+				(size 1.27 1.27)
+			)
+			(justify left)
+		)
+		(property "Intersheetrefs" "${INTERSHEET_REFS}"
+			(at 165.3865 148.59 0)
+			(effects
+				(font
+					(size 1.27 1.27)
+				)
+				(justify left)
 				(hide yes)
 			)
@@
 					(unit 1)
 				)
+			)
+		)
+	)
+	(symbol
+		(lib_id "Ts_Foc_Vo符号库:RES")
+		(at 153.67 148.59 0)
+		(unit 1)
+		(exclude_from_sim no)
+		(in_bom yes)
+		(on_board yes)
+		(dnp no)
+		(property "Reference" "R37"
+			(at 155.702 150.876 0)
+			(effects
+				(font
+					(size 1.27 1.27)
+				)
+			)
+		)
+		(property "Value" "1.5k"
+			(at 151.384 150.876 0)
+			(effects
+				(font
+					(size 1.27 1.27)
+				)
+			)
+		)
+		(property "Footprint" "Ts_Foc_Vo封装库:Res_0402"
+			(at 153.924 151.13 0)
+			(effects
+				(font
+					(size 1.27 1.27)
+				)
+				(hide yes)
+			)
+		)
+		(property "Datasheet" ""
+			(at 153.67 154.94 0)
+			(effects
+				(font
+					(size 1.27 1.27)
+				)
+				(hide yes)
+			)
+		)
+		(property "Description" ""
+			(at 153.67 148.59 0)
+			(effects
+				(font
+					(size 1.27 1.27)
+				)
+				(hide yes)
+			)
+		)
+		(property "SuppliersPartNumber" "C5200633"
+			(at 153.67 160.02 0)
+			(effects
+				(font
+					(size 1.27 1.27)
+				)
+				(hide yes)
+			)
+		)
+		(property "uuid" "std:0c78b8f437b74d4badbc2695159e48f2"
+			(at 153.67 160.02 0)
+			(effects
+				(font
+					(size 1.27 1.27)
+				)
+				(hide yes)
+			)
+		)
+		(pin "1"
+		)
+		(pin "2"
+		)
+		(instances
+			(project "Ts_Foc_Vo1_0"
+				(path "/0cbcabec-8024-48c7-ab91-86e279a5637e/f3329442-eac4-40be-b987-eebdbe922017/a35a2634-1c1b-4e39-9abf-0b7a592915e4"
+					(reference "R37")
+					(unit 1)
+				)

Commit message: 电源走线完成
Connections:
- net DM renamed DN
- net USB-DM renamed USB-DN
Changed lines of the file:
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@@
 		)
 	)
-	(global_label "DM"
+	(global_label "DN"
 		(shape bidirectional)
 		(at 148.59 95.25 180)
@@
 		)
 		(property "Intersheetrefs" "${INTERSHEET_REFS}"
-			(at 141.7721 95.25 0)
+			(at 141.893 95.25 0)
 			(effects
 				(font
@@
 		)
 	)
-	(global_label "USB-DM"
+	(global_label "USB-DN"
 		(shape bidirectional)
 		(at 148.59 130.81 180)
@@
 		)
 		(property "Intersheetrefs" "${INTERSHEET_REFS}"
-			(at 136.3897 130.81 0)
+			(at 136.5106 130.81 0)
 			(effects
 				(font
@@
 		)
 	)
-	(global_label "DM"
+	(global_label "DN"
 		(shape bidirectional)
 		(at 158.75 130.81 0)
@@
 		)
 		(property "Intersheetrefs" "${INTERSHEET_REFS}"
-			(at 165.5679 130.81 0)
+			(at 165.447 130.81 0)
 			(effects
 				(font
@@
 		)
 	)
-	(global_label "DM"
+	(global_label "DN"
 		(shape bidirectional)
 		(at 148.59 100.33 180)
@@
 		)
 		(property "Intersheetrefs" "${INTERSHEET_REFS}"
-			(at 141.7721 100.33 0)
-			(effects
-				(font
+			(at 141.893 100.33 0)
+			(effects
+				(font
