File: TsFoc/ts_foc_fw/Ts_Foc_Vesc0.1/Ts_Foc_Vesc0_1/Ts_Foc_Vo1_0.kicad_pcb (KiCad board)
At the start: 2 copper layers, 130 parts, among them CN1 MR30PW-M30.G.Y, CN10 GH1.25-4P, CN11 GH1.25-5PLT, CN12 GH1.25-5PLT, CN2 MR30PW-M30.G.Y, CN3 GH1.25-2P_LT, CN4 GH1.25-2P_LT, CN5 XT30PW-M, CN6 GH1.25-4P, CN7 GH1.25-4P, CN8 GH1.25-4P, CN9 GH1.25-4P, J1 Conn_01x04, Q1 JSM2301S, Q10 RU3089M-C, Q11 RU3089M-C, Q12 RU3089M-C, Q13 RU3089M-C, Q2 RU3089M-C, Q3 RU3089M-C, Q4 RU3089M-C, Q5 RU3089M-C, Q6 RU3089M-C, Q7 RU3089M-C, Q8 RU3089M-C, Q9 RU3089M-C, SW1 BOTTOM, SW2 BOTTOM, U1 TPS5430DDAR, U10 SIT1050TK, U11 SIT1050TK, U2 AMS1117-3.3V, U3 STM32F407VET6, U4 EG2133, U5 INA240A2PWR, U6 INA240A2PWR, U7 EG2133, U8 INA240A2PWR, U9 INA240A2PWR, X1 25Mhz

Commit message: PCB_Layout_success
Parts:
- removed CN1, CN2: MR30PW-M30.G.Y, Ts_Foc_Vo封装库:MR30PW-M30-G-Y
- removed J1: Conn_01x04, Connector_PinHeader_2.54mm:PinHeader_1x04_P2.54mm_Vertical
- added C32: 100nf, Ts_Foc_Vo封装库:CAP_0402, B.Cu at (135.1, 90.5)
- added C33: 100nf, Ts_Foc_Vo封装库:CAP_0402, B.Cu at (135.2, 91.7)
- added C34: 100nf, Ts_Foc_Vo封装库:CAP_0402, B.Cu at (109.2, 94.7)
- added C35: 100nf, Ts_Foc_Vo封装库:CAP_0402, B.Cu at (109.1, 93.5)
- added C36: 100nf, Ts_Foc_Vo封装库:CAP_0402, B.Cu at (135.2, 89.4)
- added C37: 100nf, Ts_Foc_Vo封装库:CAP_0402, B.Cu at (130.9, 91.4)
- added C38: 100nf, Ts_Foc_Vo封装库:CAP_0402, B.Cu at (129.8, 91.4)
- added C39: 100nf, Ts_Foc_Vo封装库:CAP_0402, B.Cu at (138.6, 77.5)
- added C40: 100nf, Ts_Foc_Vo封装库:CAP_0402, B.Cu at (138.7, 76.3)
- added C41: 100nf, Ts_Foc_Vo封装库:CAP_0402, B.Cu at (129.9, 71.7)
- added C42: 100nf, Ts_Foc_Vo封装库:CAP_0402, B.Cu at (131.1, 71.7)
- added CN13: GH1.25-4P, Ts_Foc_Vo封装库:GH1.25_CONN-SMD_4P-P1.25, F.Cu at (99.7, 99.7)
- added H1: MountingHole_Pad, MountingHole:MountingHole_3.7mm_Pad_Via, F.Cu at (96.6, 61.7)
- added H2: MountingHole_Pad, MountingHole:MountingHole_3.7mm_Pad_Via, F.Cu at (96.6, 118.7)
- added H3: MountingHole_Pad, MountingHole:MountingHole_3.7mm_Pad_Via, F.Cu at (156.1, 61.7)
- added H4: MountingHole_Pad, MountingHole:MountingHole_3.7mm_Pad_Via, F.Cu at (156.1, 118.6)
- added H5: MountingHole, MountingHole:MountingHole_3.2mm_M3, F.Cu at (100.3, 110.7)
- added H6: MountingHole, MountingHole:MountingHole_3.2mm_M3, F.Cu at (151.3, 68.1)
- added R37: 1.5k, Ts_Foc_Vo封装库:Res_0402, B.Cu at (150.6, 96.8)
- C10, C11, C12, C13, C14, C15, C19, C2, C20, C21, C22, C23, C24, C25, C26, C27, C28, C3, C4, C5, C6, C7, C8, C9, CN5, D12, D13, D14, D3, D4, D5, Q1, Q11, Q13, Q3, Q5, Q7, Q9, R1, R12, R13, R14, R15, R16, R2, R23, R24, R3, R33, R34, R35, R36, R5, R6, U4, U5, U6, U7, U8, U9: moved to B.Cu
- moved L1 197.9 mm to (151.9, 106.9), turned to 90 degrees
- moved C2 189.5 mm to (147.0, 99.4), turned to -90 degrees
- moved C1 186.3 mm to (141.9, 100.6), turned to 90 degrees
- moved R1 184.9 mm to (145.8, 99.5), turned to 90 degrees
- moved D1 184.1 mm to (144.7, 108.7), turned to 180 degrees
- moved C3 181.2 mm to (139.9, 97.3), turned to -90 degrees
- moved C5 179.9 mm to (138.4, 101.8)
- moved C6 179.5 mm to (138.4, 103.0)
- moved C4 179.2 mm to (138.7, 97.3), turned to -90 degrees
- moved U1 176.7 mm to (138.5, 99.7), turned to -90 degrees
- moved R2 174.8 mm to (137.1, 96.7)
- moved R3 174.3 mm to (137.0, 97.8), turned to 180 degrees
- moved USB1 164.1 mm to (151.0, 96.6), turned to 90 degrees
- moved R33 162.1 mm to (150.6, 98.4), turned to 180 degrees
- moved R34 158.3 mm to (150.6, 95.3), turned to 180 degrees
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Connections:
- C19 pad 2: Net-(U4-VCC) -> 5V
- C20 pad 2: Net-(U4-VCC) -> 5V
- C24 pad 2: Net-(U7-VCC) -> 5V
- C25 pad 2: Net-(U7-VCC) -> 5V
- C7 pad 1: 5V_DC -> 5V
- C8 pad 1: 5V_DC -> 5V
- Q1 pad 3: 5V_USB -> 5V-USB
- U2 pad 3: 5V_DC -> 5V
- U4 pad 7: Net-(U4-VCC) -> 5V
- U7 pad 7: Net-(U7-VCC) -> 5V
Routing:
- net 3V3: track 0.00 -> 65.9 mm, vias 0 -> 8
- net GND: track 0.00 -> 33.1 mm, vias 0 -> 4
- net Net-(D6-A): track 0.00 -> 10.9 mm, vias 0 -> 1
- net Net-(D19-A): track 0.00 -> 9.65 mm, vias 0 -> 1
- net ADC1-IN3: track 0.00 -> 9.25 mm, vias 0 -> 1
- net Net-(D7-A): track 0.00 -> 8.86 mm
- net Net-(D20-A): track 0.00 -> 8.68 mm
- net Net-(D8-A): track 0.00 -> 8.68 mm, vias 0 -> 3
- net ADC1-IN2: track 0.00 -> 8.66 mm, vias 0 -> 1
- net PB12: track 0.00 -> 8.63 mm
- net PE2: track 0.00 -> 8.63 mm
- net Net-(U3A-VCAP_1): track 0.00 -> 8.50 mm, vias 0 -> 1
- net ADC1-IN1: track 0.00 -> 8.50 mm, vias 0 -> 1
- net SPI2-SCK: track 0.00 -> 8.48 mm, vias 0 -> 1
- net PE3: track 0.00 -> 8.48 mm
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Other:
- board outline added: 59.4 x 56.8 mm
- copper layers 2 -> 4

Commit message: 电源走线完成
Parts:
- added R38: 0r, Ts_Foc_Vo封装库:Res_0402, F.Cu at (104.4, 103.7)
- moved C25 8.31 mm to (131.1, 79.8)
- moved C19 8.20 mm to (121.0, 79.8)
- moved C24 6.17 mm to (129.8, 79.8), turned to 90 degrees
- moved C20 5.98 mm to (119.8, 79.8), turned to 90 degrees
- moved C2 2.79 mm to (145.4, 101.7), turned to 180 degrees
- moved Q1 2.30 mm to (145.8, 99.5)
- moved R1 2.16 mm to (147.2, 101.1), turned to -90 degrees
- moved R5 1.79 mm to (143.4, 102.0)
- moved D2 0.51 mm to (143.3, 100.8)
- moved LED1 0.49 mm to (144.1, 97.8)
- moved C21 0.42 mm to (118.9, 90.5)
- moved C22 0.42 mm to (117.7, 90.4)
- moved C23 0.42 mm to (116.5, 90.4)
- moved R4 0.26 mm to (141.9, 98.0)
- moved R7 0.24 mm to (134.7, 97.2)
Connections:
- net DM renamed DN
- net USB-DM renamed USB-DN
Routing:
- net 3V3: track 65.9 -> 271.1 mm, vias 8 -> 10
- net 5V: track 0.00 -> 84.3 mm, vias 0 -> 4
- net USB-DN: track 7.89 -> 68.1 mm, vias 1 -> 2
- net USB-DP: track 8.04 -> 68.1 mm, vias 1 -> 2
- net M0_GH3: track 3.54 -> 39.8 mm, vias 0 -> 1
- net M0_GH2: track 4.94 -> 40.1 mm
- net M0_GH1: track 6.90 -> 41.3 mm, vias 0 -> 1
- net 5V_DC: track 0.00 -> 22.0 mm, vias 0 -> 1
- net NRST: track 7.32 -> 28.0 mm, vias 1 -> 2
- net PH: track 0.00 -> 19.5 mm
- net SWCLK: track 0.00 -> 17.7 mm
- net SWDIO: track 8.20 -> 21.8 mm, vias 1 -> 3
- net Net-(U3A-BOOT0): track 0.00 -> 12.1 mm, vias 0 -> 2
- net Net-(D5-K): track 0.00 -> 11.7 mm, vias 0 -> 2
- net Net-(D4-K): track 0.00 -> 11.5 mm, vias 0 -> 2
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- added copper zone on F.Cu, net VCC

Commit message: 第一版layout完成，准备打板验证
Parts:
- added CN14: ~, Ts_Foc_Vo封装库:通孔焊盘, F.Cu at (103.1, 114.0)
- added CN15: ~, Ts_Foc_Vo封装库:通孔焊盘, F.Cu at (108.5, 114.0)
- added CN16: ~, Ts_Foc_Vo封装库:通孔焊盘, F.Cu at (113.8, 114.0)
- added CN17: ~, Ts_Foc_Vo封装库:通孔焊盘, F.Cu at (119.2, 114.0)
- added CN18: ~, Ts_Foc_Vo封装库:通孔焊盘, F.Cu at (124.5, 114.0)
- added CN19: ~, Ts_Foc_Vo封装库:通孔焊盘, F.Cu at (129.8, 114.0)
- R38, R4, R9: moved to B.Cu
- moved U5 31.9 mm to (107.4, 100.3), turned to 180 degrees
- moved U6 25.6 mm to (115.7, 100.4), turned to 180 degrees
- moved R13 25.2 mm to (144.1, 69.0), turned to 180 degrees
- moved C10 25.1 mm to (137.2, 65.6), turned to 0 degrees
- moved R4 24.7 mm to (143.0, 73.4), turned to 180 degrees
- moved LED1 24.5 mm to (143.0, 73.4), turned to 0 degrees
- moved C9 23.6 mm to (137.2, 66.8), turned to 0 degrees
- moved LED2 23.6 mm to (143.0, 71.7)
- moved U9 23.4 mm to (132.4, 100.3), turned to 180 degrees
- moved LED3 23.3 mm to (142.9, 69.6), turned to 180 degrees
- moved R9 23.2 mm to (143.0, 71.7), turned to 180 degrees
- moved R14 22.9 mm to (144.2, 70.1), turned to 180 degrees
- moved R12 22.7 mm to (141.5, 69.1)
- moved C7 21.7 mm to (139.7, 72.0), turned to 0 degrees
- moved U2 20.7 mm to (137.8, 71.3), turned to -90 degrees
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Connections:
- net FDCAN1-H renamed FDCAN1+
- net FDCAN1-L renamed FDCAN1-
- net FDCAN2-H renamed FDCAN2+
- net FDCAN2-L renamed FDCAN2-
Routing:
- net GND: track 36.3 -> 124.6 mm, vias 26 -> 172
- net VCC: track 6.24 -> 89.1 mm, vias 0 -> 4
- net ADC1-IN0: track 8.35 -> 61.4 mm, vias 1 -> 2
- net ADC1-IN1: track 8.50 -> 55.4 mm, vias 1 -> 2
- net FDCAN1-TX: track 0.00 -> 42.1 mm, vias 0 -> 2
- net ADC1-IN2: track 8.66 -> 48.5 mm, vias 1 -> 2
- net PGND: track 0.00 -> 39.7 mm
- net 3V3: track 271.1 -> 309.5 mm, vias 10 -> 14
- net M1_OUT3: track 2.99 -> 39.9 mm, vias 1 -> 3
- net ADC1-IN3: track 9.25 -> 44.3 mm, vias 1 -> 2
- net FDCAN1-RX: track 0.00 -> 33.1 mm, vias 0 -> 2
- net I2C1-SCL: track 0.00 -> 32.0 mm, vias 0 -> 2
- net RGB-B: track 7.77 -> 39.4 mm, vias 1 -> 2
- net 5V: track 84.3 -> 115.5 mm
- net I2C1-SDA: track 0.00 -> 28.7 mm, vias 0 -> 2
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- added copper zone on B.Cu, net GND
- added copper zone on F.Cu, net GND
- added copper zone on In1.Cu, net GND
- added copper zone on In2.Cu, net GND
Other:
- board size 59.4 x 56.8 mm -> 55.8 x 56.8 mm
- board text added: "3V3"
- board text added: "BT"
- board text added: "CAN1"
- board text added: "CAN2"
- board text added: "CLK"
- board text added: "DIO"
- board text added: "GND"
- board text added: "H"
- board text added: "IIC1"
- board text added: "IIC2"
- board text added: "L"
- board text added: "MISO"
- board text added: "MOSI"
- board text added: "RX"
- board text added: "SCK"
- board text added: "SCL"
- board text added: "SDA"
- board text added: "SPI1"
- board text added: "SPI2"
- board text added: "SWD"
- board text added: "TX"
- board text added: "UART1"
- board text added: "UART2"
- board text added: "UART3"
- board text added: "_________"
