File: TsFoc/ts_foc_fw/Ts_Foc_Vesc0.2/Ts_Foc_Vesc0_2/Ts_Foc_Vo1_0.kicad_pcb (KiCad board)
At the start: 4 copper layers, 55.8 x 56.8 mm, 152 parts, among them CN10 GH1.25-4P, CN11 GH1.25-5PLT, CN12 GH1.25-5PLT, CN13 GH1.25-4P, CN3 GH1.25-2P_LT, CN4 GH1.25-2P_LT, CN5 XT30PW-M, CN6 GH1.25-4P, CN7 GH1.25-4P, CN8 GH1.25-4P, CN9 GH1.25-4P, Q1 JSM2301S, Q10 RU3089M-C, Q11 RU3089M-C, Q12 RU3089M-C, Q13 RU3089M-C, Q2 RU3089M-C, Q3 RU3089M-C, Q4 RU3089M-C, Q5 RU3089M-C, Q6 RU3089M-C, Q7 RU3089M-C, Q8 RU3089M-C, Q9 RU3089M-C, SW1 BOTTOM, SW2 BOTTOM, U1 TPS5430DDAR, U10 SIT1050TK, U11 SIT1050TK, U2 AMS1117-3.3V, U3 STM32F407VET6, U4 EG2133, U5 INA240A2PWR, U6 INA240A2PWR, U7 EG2133, U8 INA240A2PWR, U9 INA240A2PWR, X1 25Mhz

Commit message: 1. can通信测试通过 2. as5600通信测试通过 3. PCB板桥驱动电路有标签错误，导致有四个引脚未能链接 4.
Parts:
- C18: value 22pf -> 100nf
Connections:
- C21 pad 1: M0_OUT1 -> M0_OUT1_P
- C22 pad 1: M0_OUT2 -> M0_OUT2_P
- C26 pad 1: M1_OUT1 -> M1_OUT1_P
- C27 pad 1: M1_OUT2 -> M1_OUT2_P
- U4 pad 15: M0_OUT2 -> M0_OUT2_P
- U4 pad 18: M0_OUT1 -> M0_OUT1_P
- U7 pad 15: M1_OUT2 -> M1_OUT2_P
- U7 pad 18: M1_OUT1 -> M1_OUT1_P
Routing:
- net M0_OUT1: track 9.56 -> 0.00 mm
- net M0_OUT1_P: track 16.6 -> 26.2 mm
- net M1_OUT1: track 9.48 -> 0.00 mm
- net M1_OUT1_P: track 15.5 -> 25.0 mm
- net M0_OUT2_P: track 19.2 -> 26.3 mm
- net M0_OUT2: track 7.10 -> 0.00 mm
- net M1_OUT2_P: track 18.1 -> 24.8 mm
- net M1_OUT2: track 6.64 -> 0.00 mm
